File: Hitodama-valves-board.sch (KiCad schematic (older format))
At the start: 33 parts, among them J1 Solenoid A, J10 PWMB, J11 STANDBY, J2 Solenoid B, J3 Pressure_amp_b, J4 Pressure_amp_a, J5 PWMA, J6 AIN2, J7 AIN1, J8 BIN1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

Commit message: improved adding +12v connector
Parts:
- added J12: +12v_SUPPLY, Connector_Pin:Pin_D1.0mm_L10.0mm_LooseFit, symbol Connector:Conn_01x01_Female
Changed lines of the file:
@@
 	1    0    0    -1
 $EndComp
+$Comp
+L Connector:Conn_01x01_Female J12
+U 1 1 5CB626E2
+P 6200 6200
+F 0 "J12" H 6227 6226 50  0000 L CNN
+F 1 "+12v_SUPPLY" H 6350 6200 50  0000 L CNN
+F 2 "Connector_Pin:Pin_D1.0mm_L10.0mm_LooseFit" H 6200 6200 50  0001 C CNN
+F 3 "~" H 6200 6200 50  0001 C CNN
+	1    6200 6200
+	1    0    0    -1
+$EndComp
+$Comp
+L power:+12V #PWR0115
+U 1 1 5CB628B6
+P 6000 6200
+F 0 "#PWR0115" H 6000 6050 50  0001 C CNN
+F 1 "+12V" V 6015 6328 50  0000 L CNN
+F 2 "" H 6000 6200 50  0001 C CNN
+F 3 "" H 6000 6200 50  0001 C CNN
+	1    6000 6200
+	0    -1   -1   0
+$EndComp
 $EndSCHEMATC

Commit message: changed design rules for milling machine and consequently re-routed everyhting
Parts:
- added J13: VCC supply, Connector_Pin:Pin_D1.0mm_L10.0mm_LooseFit, symbol Connector:Conn_01x01_Female
- added J14: GND, Connector_Pin:Pin_D1.0mm_L10.0mm_LooseFit, symbol Connector:Conn_01x01_Female
- JP1: footprint Jumper:SolderJumper-2_P1.3mm_Bridged_Pad1.0x1.5mm -> Jumper:SolderJumper-2_P1.3mm_Bridged2Bar_Pad1.0x1.5mm
Other:
- moved on the sheet: H1, H2, H3, H4
Changed lines of the file:
@@
 F 0 "JP1" H 5300 5100 50  0000 C CNN
 F 1 "(A,B)IN 1" H 5050 5100 50  0000 C CNN
-F 2 "Jumper:SolderJumper-2_P1.3mm_Bridged_Pad1.0x1.5mm" H 5050 5200 50  0001 C CNN
+F 2 "Jumper:SolderJumper-2_P1.3mm_Bridged2Bar_Pad1.0x1.5mm" H 5050 5200 50  0001 C CNN
 F 3 "~" H 5050 5200 50  0001 C CNN
 	1    5050 5200
@@
 L Mechanical:MountingHole H1
 U 1 1 5CB701BB
-P 6000 6500
-F 0 "H1" H 6100 6546 50  0000 L CNN
-F 1 "MountingHole" H 6100 6455 50  0000 L CNN
-F 2 "MountingHole:MountingHole_3.2mm_M3" H 6000 6500 50  0001 C CNN
-F 3 "~" H 6000 6500 50  0001 C CNN
-	1    6000 6500
+P 6000 7050
+F 0 "H1" H 6100 7096 50  0000 L CNN
+F 1 "MountingHole" H 6100 7005 50  0000 L CNN
+F 2 "MountingHole:MountingHole_3.2mm_M3" H 6000 7050 50  0001 C CNN
+F 3 "~" H 6000 7050 50  0001 C CNN
+	1    6000 7050
 	1    0    0    -1
 $EndComp
@@
 L Mechanical:MountingHole H2
 U 1 1 5CB704E4
-P 6000 6700
-F 0 "H2" H 6100 6746 50  0000 L CNN
-F 1 "MountingHole" H 6100 6655 50  0000 L CNN
-F 2 "MountingHole:MountingHole_3.2mm_M3" H 6000 6700 50  0001 C CNN
-F 3 "~" H 6000 6700 50  0001 C CNN
-	1    6000 6700
+P 6000 7250
+F 0 "H2" H 6100 7296 50  0000 L CNN
+F 1 "MountingHole" H 6100 7205 50  0000 L CNN
+F 2 "MountingHole:MountingHole_3.2mm_M3" H 6000 7250 50  0001 C CNN
+F 3 "~" H 6000 7250 50  0001 C CNN
+	1    6000 7250
 	1    0    0    -1
 $EndComp
@@
 L Mechanical:MountingHole H3
 U 1 1 5CB70540
-P 6000 6900
-F 0 "H3" H 6100 6946 50  0000 L CNN
-F 1 "MountingHole" H 6100 6855 50  0000 L CNN
-F 2 "MountingHole:MountingHole_3.2mm_M3" H 6000 6900 50  0001 C CNN
-F 3 "~" H 6000 6900 50  0001 C CNN
-	1    6000 6900
+P 6000 7450
+F 0 "H3" H 6100 7496 50  0000 L CNN
+F 1 "MountingHole" H 6100 7405 50  0000 L CNN
+F 2 "MountingHole:MountingHole_3.2mm_M3" H 6000 7450 50  0001 C CNN
+F 3 "~" H 6000 7450 50  0001 C CNN
+	1    6000 7450
 	1    0    0    -1
 $EndComp
@@
 L Mechanical:MountingHole H4
 U 1 1 5CB70598
-P 6000 7100
-F 0 "H4" H 6100 7146 50  0000 L CNN
-F 1 "MountingHole" H 6100 7055 50  0000 L CNN
-F 2 "MountingHole:MountingHole_3.2mm_M3" H 6000 7100 50  0001 C CNN
-F 3 "~" H 6000 7100 50  0001 C CNN
-	1    6000 7100
+P 6000 7650
+F 0 "H4" H 6100 7696 50  0000 L CNN
+F 1 "MountingHole" H 6100 7605 50  0000 L CNN
+F 2 "MountingHole:MountingHole_3.2mm_M3" H 6000 7650 50  0001 C CNN
+F 3 "~" H 6000 7650 50  0001 C CNN
+	1    6000 7650
 	1    0    0    -1
 $EndComp
@@
 	0    -1   -1   0
 $EndComp
+$Comp
+L Connector:Conn_01x01_Female J13
+U 1 1 5CB734CF
+P 6200 6350
+F 0 "J13" H 6227 6376 50  0000 L CNN
+F 1 "VCC supply" H 6350 6350 50  0000 L CNN
+F 2 "Connector_Pin:Pin_D1.0mm_L10.0mm_LooseFit" H 6200 6350 50  0001 C CNN
+F 3 "~" H 6200 6350 50  0001 C CNN
+	1    6200 6350
+	1    0    0    -1
+$EndComp
+$Comp
+L Connector:Conn_01x01_Female J14
+U 1 1 5CB76CD1
+P 6200 6500
+F 0 "J14" H 6227 6526 50  0000 L CNN
+F 1 "GND" H 6350 6500 50  0000 L CNN
+F 2 "Connector_Pin:Pin_D1.0mm_L10.0mm_LooseFit" H 6200 6500 50  0001 C CNN
+F 3 "~" H 6200 6500 50  0001 C CNN
+	1    6200 6500
+	1    0    0    -1
+$EndComp
+$Comp
+L power:VCC #PWR0116
+U 1 1 5CB789A0
+P 6000 6350
+F 0 "#PWR0116" H 6000 6200 50  0001 C CNN
+F 1 "VCC" V 6018 6477 50  0000 L CNN
+F 2 "" H 6000 6350 50  0001 C CNN
+F 3 "" H 6000 6350 50  0001 C CNN
+	1    6000 6350
+	0    -1   -1   0
+$EndComp
+$Comp
+L power:GND #PWR0117
+U 1 1 5CB78A95
+P 6000 6500
+F 0 "#PWR0117" H 6000 6250 50  0001 C CNN
+F 1 "GND" H 6005 6327 50  0000 C CNN
+F 2 "" H 6000 6500 50  0001 C CNN
+F 3 "" H 6000 6500 50  0001 C CNN
+	1    6000 6500
+	1    0    0    -1
+$EndComp
 $EndSCHEMATC
