File: Hitodama-valve-boards.sch (KiCad schematic (older format))
At the start: 25 parts, among them J1 Solenoid A, J2 Solenoid B, U1 LM358, U2 Pressure_b, U3 Pressure_a, U4 ChamberBoard_Holder, U5 Pololu-713

Commit message: change connectors into edge connector 5-5530843-3, TE Connectivity
Parts:
- U4: footprint chamber_board_holder:chamber_board_holder -> chamber_board_holder:chamber_board_holder_ 5-5530843-3_male
Changed lines of the file:
@@
 F 0 "U4" H 8069 3411 50  0000 L CNN
 F 1 "ChamberBoard_Holder" H 8069 3320 50  0000 L CNN
-F 2 "chamber_board_holder:chamber_board_holder" H 7400 3450 50  0001 C CNN
+F 2 "chamber_board_holder:chamber_board_holder_ 5-5530843-3_male" H 7400 3450 50  0001 C CNN
 F 3 "" H 7400 3450 50  0001 C CNN
 	1    7400 3450
