File: Hitodama-teensy-board.kicad_pcb (KiCad board)
At the start: 2 copper layers, 101.6 x 127 mm, 16 parts, among them J1 Jack-DC, J2 Conn_01x20_Female, J3 Conn_01x20_Female, J4 Conn_01x20_Female, U4 Teensy3.6

Commit message: 2 row connector, routed on intermediate board
Parts:
- J2, J3, J4: footprint Connector_PinHeader_2.54mm:PinHeader_1x20_P2.54mm_Vertical -> Connector_IDC:IDC-Header_2x10_P2.54mm_Vertical
- moved U4 17.8 mm to (71.1, 45.8)
- moved J2 9.36 mm to (24.5, 79.2)
- moved J3 9.36 mm to (53.7, 79.2)
- moved J4 9.36 mm to (82.9, 79.2)
Routing:
- net GND: track 240.2 -> 0.00 mm
- net VCC: track 204.0 -> 0.00 mm
- net /All.Stby: track 202.7 -> 0.00 mm
- net /ChamberH.ADC: track 183.0 -> 0.00 mm, vias 1 -> 0
- net /ChamberI.ADC: track 123.1 -> 0.00 mm, vias 1 -> 0
- net /ChamberI.D2: track 121.5 -> 0.00 mm, vias 1 -> 0
- net /ChamberC.PWM: track 119.1 -> 0.00 mm
- net /ChamberB.PWM: track 109.1 -> 0.00 mm
- net /ChamberH.D1: track 96.9 -> 0.00 mm
- net /ChamberG.ADC: track 96.2 -> 0.00 mm, vias 2 -> 0
- net /SPI0.SCK: track 93.7 -> 0.00 mm
- net /ChamberH.D2: track 91.4 -> 0.00 mm
- net /ChamberH.D3: track 90.8 -> 0.00 mm
- net /ChamberA.D1: track 88.1 -> 0.00 mm
- net /SPI0.MISO: track 86.1 -> 0.00 mm
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- added copper zone on B.Cu, net GND
- added copper zone on F.Cu, net GND
